File: tests/fixtures/MicrasMainBoard.kicad_pcb (KiCad board)
At the start: 154 parts

Commit message: ✨ Quote a whole JLCPCB order, the boards priced live from the KiCad board plus their assembly
Parts:
- removed the ? at (0.00, 0.00) (x4)
- added ? (x4): , , B.Cu at (0.00, 0.00)
- 20V, BZ1, C1, C10, C11, C12, C13, C14, C15, C16, C17, C18, C19, C2, C20, C21, C22, C23, C24, C25, C26, C27, C28, C29, C3, C30, C31, C32, C33, C34, C35, C36, C37, C38, C39, C4, C40, C41, C42, C43, C44, C45, C46, C47, C48, C49, C5, C50, C51, C52, C53, C54, C55, C56, C57, C6, C60, C7, C8, C9, D1, D2, D3, D4, D5, D6, D7, EC1, EC2, F1, FAN_ENABLE, FAN_OVERCURRENT, FAN_PWM, IC1, IC2, IC3, IC4, IC5, IC6, IC7, IMU_INT1, IMU_INT2, J1, L1, L2, L3, M1, M2, M3, P1, Q1, Q2, Q3, Q4, Q5, Q6, R1, R10, R11, R12, R13, R14, R15, R16, R17, R18, R19, R2, R20, R21, R22, R23, R24, R25, R26, R27, R28, R29, R3, R30, R31, R32, R33, R34, R35, R36, R37, R38, R39, R4, R40, R41, R42, R5, R6, R7, R8, R9, SW1, SW2, SW3, SW4, SW5, U1, U2, U3, W1, W2, W3, W4: moved to B.Cu
Other:
- board outline added: 50 x 90 mm
- copper layers 0 -> 4
Changed lines of the file:
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@@
 (kicad_pcb
+	(general
+		(thickness 1.0412)
+		(legacy_teardrops no)
+	)
+	(layers
+		(0 "F.Cu" signal "Top Layer")
+		(4 "In1.Cu" signal "Inner Layer 1")
+		(6 "In2.Cu" signal "Inner Layer 2")
+		(2 "B.Cu" signal "Bottom Layer")
+		(9 "F.Adhes" user "F.Adhesive")
+		(11 "B.Adhes" user "B.Adhesive")
+		(13 "F.Paste" user "Top Paste")
+		(15 "B.Paste" user "Bottom Paste")
+		(5 "F.SilkS" user "Top Overlay")
+		(7 "B.SilkS" user "Bottom Overlay")
+		(1 "F.Mask" user "Top Solder")
+		(3 "B.Mask" user "Bottom Solder")
+		(17 "Dwgs.User" user "User.Drawings")
+		(19 "Cmts.User" user "User.Comments")
+		(21 "Eco1.User" user "User.Eco1")
+		(23 "Eco2.User" user "User.Eco2")
+		(25 "Edge.Cuts" user)
+		(27 "Margin" user)
+		(31 "F.CrtYd" user "Top Courtyard")
+		(29 "B.CrtYd" user "Bottom Courtyard")
+		(35 "F.Fab" user "Top Component Center")
+		(33 "B.Fab" user "Bottom Component Center")
+		(39 "User.1" user "Mechanical 1")
+		(41 "User.2" user)
+		(43 "User.3" user)
+		(45 "User.4" user)
+		(53 "User.8" user "Top 3D Body")
+		(55 "User.9" user "Bottom 3D Body")
+		(63 "User.13" user "Mechanical 13")
+		(67 "User.15" user "Mechanical 15")
+	)
+	(gr_line (start 123.501095 81.183943) (end 123.501105 81.18394) (layer "Edge.Cuts"))
+	(gr_arc (start 123.501095 81.183943) (mid 123.634841 80.035174) (end 124.028961 78.947873) (layer "Edge.Cuts"))
+	(gr_line (start 123.501105 81.18394) (end 123.501105 103.0036) (layer "Edge.Cuts"))
+	(gr_line (start 123.501105 124.0036) (end 123.501105 148.0036) (layer "Edge.Cuts"))
+	(gr_arc (start 123.501105 124.0036) (mid 124.086891 122.589386) (end 125.501105 122.0036) (layer "Edge.Cuts"))
+	(gr_arc (start 125.501105 105.0036) (mid 124.086891 104.417814) (end 123.501105 103.0036) (layer "Edge.Cuts"))
+	(gr_line (start 125.501105 105.0036) (end 129.251104 105.0036) (layer "Edge.Cuts"))
+	(gr_arc (start 125.501105 150.0036) (mid 124.086891 149.417814) (end 123.501105 148.0036) (layer "Edge.Cuts"))
+	(gr_line (start 125.501105 150.0036) (end 144.451105 150.0036) (layer "Edge.Cuts"))
+	(gr_arc (start 129.251104 105.0036) (mid 130.665318 105.589386) (end 131.251105 107.003599) (layer "Edge.Cuts"))
+	(gr_line (start 129.251105 122.0036) (end 125.501105 122.0036) (layer "Edge.Cuts"))
+	(gr_line (start 129.251106 122.0036) (end 129.251105 122.0036) (layer "Edge.Cuts"))
+	(gr_line (start 131.251105 107.003599) (end 131.251105 107.0036) (layer "Edge.Cuts"))
+	(gr_line (start 131.251105 107.0036) (end 131.251105 120.003599) (layer "Edge.Cuts"))
+	(gr_arc (start 131.251105 120.003599) (mid 130.665319 121.417813) (end 129.251106 122.0036) (layer "Edge.Cuts"))
+	(gr_line (start 132.810115 61.38556) (end 124.028961 78.947873) (layer "Edge.Cuts"))
+	(gr_line (start 132.810124 61.385565) (end 132.810115 61.38556) (layer "Edge.Cuts"))
+	(gr_arc (start 132.810124 61.385565) (mid 133.731863 60.376968) (end 135.046191 60.0036) (layer "Edge.Cuts"))
+	(gr_arc (start 141.001015 96.00363) (mid 143.197714 90.700329) (end 148.501015 88.50363) (layer "Edge.Cuts"))
+	(gr_line (start 141.151105 110.9536) (end 141.151105 116.0536) (layer "Edge.Cuts"))
+	(gr_line (start 141.151105 116.0536) (end 142.051105 116.0536) (layer "Edge.Cuts"))
+	(gr_line (start 142.051105 110.9536) (end 141.151105 110.9536) (layer "Edge.Cuts"))
+	(gr_line (start 142.051105 116.0536) (end 142.051105 110.9536) (layer "Edge.Cuts"))
+	(gr_arc (start 145.251105 148.4036) (mid 145.48542 147.837915) (end 146.051105 147.6036) (layer "Edge.Cuts"))
+	(gr_arc (start 145.251105 149.2036) (mid 145.01679 149.769285) (end 144.451105 150.0036) (layer "Edge.Cuts"))
+	(gr_line (start 145.251105 149.2036) (end 145.251105 148.4036) (layer "Edge.Cuts"))
+	(gr_line (start 146.051105 147.6036) (end 154.451105 147.6036) (layer "Edge.Cuts"))
+	(gr_line (start 147.026135 138.87984) (end 147.075615 138.76039) (layer "Edge.Cuts"))
+	(gr_line (start 147.026135 138.94448) (end 147.026135 138.87984) (layer "Edge.Cuts"))
+	(gr_line (start 147.026135 139.00913) (end 147.026135 138.94448) (layer "Edge.Cuts"))
+	(gr_line (start 147.075615 138.76039) (end 147.167035 138.66897) (layer "Edge.Cuts"))
+	(gr_line (start 147.075615 139.12858) (end 147.026135 139.00913) (layer "Edge.Cuts"))
+	(gr_line (start 147.167035 138.66897) (end 147.286485 138.61949) (layer "Edge.Cuts"))
+	(gr_line (start 147.167035 139.22) (end 147.075615 139.12858) (layer "Edge.Cuts"))
+	(gr_line (start 147.286485 138.61949) (end 147.415765 138.61949) (layer "Edge.Cuts"))
+	(gr_line (start 147.286485 139.26948) (end 147.167035 139.22) (layer "Edge.Cuts"))
+	(gr_line (start 147.415765 138.61949) (end 147.535215 138.66897) (layer "Edge.Cuts"))
+	(gr_line (start 147.415765 139.26948) (end 147.286485 139.26948) (layer "Edge.Cuts"))
+	(gr_line (start 147.535215 138.66897) (end 147.626645 138.76039) (layer "Edge.Cuts"))
+	(gr_line (start 147.535215 139.22) (end 147.415765 139.26948) (layer "Edge.Cuts"))
+	(gr_line (start 147.626645 138.76039) (end 147.676115 138.87984) (layer "Edge.Cuts"))
+	(gr_line (start 147.626645 139.12858) (end 147.535215 139.22) (layer "Edge.Cuts"))
+	(gr_line (start 147.676115 138.87984) (end 147.676115 138.94448) (layer "Edge.Cuts"))
+	(gr_line (start 147.676115 138.94448) (end 147.676115 139.00913) (layer "Edge.Cuts"))
+	(gr_line (start 147.676115 139.00913) (end 147.626645 139.12858) (layer "Edge.Cuts"))
+	(gr_arc (start 148.501015 88.50363) (mid 153.804316 90.700329) (end 156.001015 96.00363) (layer "Edge.Cuts"))
+	(gr_arc (start 148.501015 103.50363) (mid 143.197714 101.306931) (end 141.001015 96.00363) (layer "Edge.Cuts"))
+	(gr_line (start 152.816065 138.87984) (end 152.865545 138.76039) (layer "Edge.Cuts"))
+	(gr_line (start 152.816065 138.94448) (end 152.816065 138.87984) (layer "Edge.Cuts"))
+	(gr_line (start 152.816065 139.00913) (end 152.816065 138.94448) (layer "Edge.Cuts"))
+	(gr_line (start 152.865545 138.76039) (end 152.956965 138.66897) (layer "Edge.Cuts"))
+	(gr_line (start 152.865545 139.12858) (end 152.816065 139.00913) (layer "Edge.Cuts"))
+	(gr_line (start 152.956965 138.66897) (end 153.076415 138.61949) (layer "Edge.Cuts"))
+	(gr_line (start 152.956965 139.22) (end 152.865545 139.12858) (layer "Edge.Cuts"))
+	(gr_line (start 153.076415 138.61949) (end 153.205695 138.61949) (layer "Edge.Cuts"))
+	(gr_line (start 153.076415 139.26948) (end 152.956965 139.22) (layer "Edge.Cuts"))
+	(gr_line (start 153.205695 138.61949) (end 153.325145 138.66897) (layer "Edge.Cuts"))
+	(gr_line (start 153.205695 139.26948) (end 153.076415 139.26948) (layer "Edge.Cuts"))
+	(gr_line (start 153.325145 138.66897) (end 153.416575 138.76039) (layer "Edge.Cuts"))
+	(gr_line (start 153.325145 139.22) (end 153.205695 139.26948) (layer "Edge.Cuts"))
+	(gr_line (start 153.416575 138.76039) (end 153.466045 138.87984) (layer "Edge.Cuts"))
+	(gr_line (start 153.416575 139.12858) (end 153.325145 139.22) (layer "Edge.Cuts"))
+	(gr_line (start 153.466045 138.87984) (end 153.466045 138.94448) (layer "Edge.Cuts"))
+	(gr_line (start 153.466045 138.94448) (end 153.466045 139.00913) (layer "Edge.Cuts"))
+	(gr_line (start 153.466045 139.00913) (end 153.416575 139.12858) (layer "Edge.Cuts"))
+	(gr_arc (start 154.451105 147.6036) (mid 155.01679 147.837915) (end 155.251105 148.4036) (layer "Edge.Cuts"))
+	(gr_line (start 154.951105 110.9536) (end 154.951105 116.0536) (layer "Edge.Cuts"))
+	(gr_line (start 154.951105 116.0536) (end 155.851105 116.0536) (layer "Edge.Cuts"))
+	(gr_line (start 155.251105 148.4036) (end 155.251105 149.2036) (layer "Edge.Cuts"))
+	(gr_line (start 155.851105 110.9536) (end 154.951105 110.9536) (layer "Edge.Cuts"))
+	(gr_line (start 155.851105 116.0536) (end 155.851105 110.9536) (layer "Edge.Cuts"))
+	(gr_arc (start 156.001015 96.00363) (mid 153.804316 101.306931) (end 148.501015 103.50363) (layer "Edge.Cuts"))
+	(gr_arc (start 156.051105 150.0036) (mid 155.48542 149.769285) (end 155.251105 149.2036) (layer "Edge.Cuts"))
+	(gr_line (start 156.051105 150.0036) (end 164.201105 150.0036) (layer "Edge.Cuts"))
+	(gr_line (start 161.956025 60.0036) (end 135.046191 60.0036) (layer "Edge.Cuts"))
+	(gr_arc (start 161.956025 60.0036) (mid 163.270346 60.376981) (end 164.192094 61.385568) (layer "Edge.Cuts"))
+	(gr_arc (start 165.001105 146.7036) (mid 165.23542 146.137915) (end 165.801105 145.9036) (layer "Edge.Cuts"))
+	(gr_arc (start 165.001105 149.2036) (mid 164.76679 149.769285) (end 164.201105 150.0036) (layer "Edge.Cuts"))
+	(gr_line (start 165.001105 149.2036) (end 165.001105 146.7036) (layer "Edge.Cuts"))
+	(gr_arc (start 165.751105 107.003601) (mid 166.336891 105.589387) (end 167.751104 105.0036) (layer "Edge.Cuts"))
+	(gr_line (start 165.751105 120.0036) (end 165.751105 107.003601) (layer "Edge.Cuts"))
+	(gr_line (start 165.801105 145.9036) (end 172.701105 145.9036) (layer "Edge.Cuts"))
+	(gr_line (start 167.751104 105.0036) (end 167.751105 105.0036) (layer "Edge.Cuts"))
+	(gr_line (start 167.751105 105.0036) (end 171.501105 105.0036) (layer "Edge.Cuts"))
+	(gr_arc (start 167.751105 122.0036) (mid 166.336891 121.417814) (end 165.751105 120.0036) (layer "Edge.Cuts"))
+	(gr_line (start 171.501105 122.0036) (end 167.751105 122.0036) (layer "Edge.Cuts"))
+	(gr_arc (start 171.501105 122.0036) (mid 172.915319 122.589386) (end 173.501105 124.0036) (layer "Edge.Cuts"))
+	(gr_line (start 172.973242 78.947874) (end 172.973245 78.94787) (layer "Edge.Cuts"))
+	(gr_arc (start 172.973242 78.947874) (mid 173.367342 80.035179) (end 173.501105 81.183943) (layer "Edge.Cuts"))
+	(gr_line (start 172.973245 78.94787) (end 164.192094 61.385568) (layer "Edge.Cuts"))
+	(gr_arc (start 173.501105 103.0036) (mid 172.915319 104.417814) (end 171.501105 105.0036) (layer "Edge.Cuts"))
+	(gr_line (start 173.501105 103.0036) (end 173.501105 81.183943) (layer "Edge.Cuts"))
+	(gr_arc (start 173.501105 145.1036) (mid 173.26679 145.669285) (end 172.701105 145.9036) (layer "Edge.Cuts"))
+	(gr_line (start 173.501105 145.1036) (end 173.501105 124.0036) (layer "Edge.Cuts"))
 	(footprint "MicrasLib:C0402"
 		(layer "F.Cu")
